File: hardware/charge_controller/charge_controller.sch (KiCad schematic (older format))
At the start: 24 parts

Commit message: auto push run at Wed Feb  3 20:24:40 EST 2021
Parts:
- added H1, H2, H3, H4: MountingHole, MountingHole:MountingHole_3.2mm_M3_Pad, symbol Mechanical:MountingHole
- D1: renamed from D?; value LED -> Red; footprint (none) -> LED_SMD:LED_0805_2012Metric; Item Cost (none) -> 0.18; MFN (none) -> 150080RS75000; Supplier (none) -> Digi-Key; Supplier P/N (none) -> 732-4984-1-ND
- D4: renamed from D?; footprint (none) -> LED_SMD:LED_0805_2012Metric; Item Cost (none) -> 0.18; MFN (none) -> 150080VS75000; Supplier (none) -> Digi-Key; Supplier P/N (none) -> 732-4986-1-ND
- D5: renamed from D?; footprint (none) -> Diode_THT:D_DO-27_P15.24mm_Horizontal; Item Cost (none) -> 0.76; MFN (none) -> 80SQ045NRLG; Supplier (none) -> Digi-Key; Supplier P/N (none) -> 80SQ045NRLGOSCT-ND
- J1, J2: renamed from J?; footprint (none) -> Connector_PinSocket_2.54mm:PinSocket_1x02_P2.54mm_Vertical
- Q1, Q2, Q3: renamed from Q?; footprint (none) -> Package_TO_SOT_THT:TO-92; symbol Device:Q_NPN_BCE -> Device:Q_NPN_EBC; Item Cost (none) -> 0.18; MFN (none) -> 2N3904-AP; Supplier (none) -> Digi-Key; Supplier P/N (none) -> 2N3904-APCT-ND
- Q4: renamed from Q?; symbol Device:Q_NMOS_SGD -> Device:Q_NMOS_GDS
- RV1: renamed from RV?; footprint (none) -> Potentiometer_THT:Potentiometer_Bourns_3299Y_Vertical; Item Cost (none) -> 2.08; MFN (none) -> PV37W103C01B00; Supplier (none) -> Digi-Key; Supplier P/N (none) -> 490-2970-ND
- gave numbers to parts that had none: 14
Connections:
- net GND: now also Q1.2 (B); no longer Q1.1 (B)
- net at C1.1, J1.1 (Pin_1), R1.1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: now also Q4.3 (S); no longer Q4.1 (S)
- net at D4.1 (K), D5.2 (A): now also Q4.2 (D); no longer Q4.3 (D)
- net at D3.2 (A): now also Q1.1 (E); no longer Q1.3 (E)
- net at C2.1, R3.2: now also Q1.3 (C), Q2.2 (B); no longer Q1.2 (C), Q2.1 (B)
- net at C2.2, R4.2: now also Q2.3 (C), Q4.1 (G); no longer Q2.2 (C), Q4.2 (G)
- net at Q3.1 (E): now also Q2.1 (E), R5.1; no longer R8.2
- net at Q3.2 (B): now also R8.2; no longer R6.2
- new net: Q3.3 (C), R6.2
